File: cad/ecad/love-letters.kicad_pcb (KiCad board)
At the start: 2 copper layers, 83 x 29 mm, 39 parts, among them J1 XF2M-2415-1A, J2 Battery Connector, Q1 BSS138, Q2 SS8050, Q3 AO3401A, SW1 SW_SPDT, U1 XIAO-ESP32-S3-SMD, U2 RT9193-33GB, U3 TXB0108PW

Commit message: Ordered Revision: Digikey and JLCPCB
Routing:
- net 3V3_OUT: track 47.9 -> 62.3 mm, vias 4 -> 5
- net GND: track 341.0 -> 355.2 mm
Other:
- board text added: "for: carol by: caleb"
- board text added: "love-letters driver board"
